File: src/pcb/omnicontroller.kicad_pcb (KiCad board)
At the start: 2 copper layers, 124.5 x 68.6 mm, 53 parts, among them J1 G-Switch GT-USB-7010ASV, J2 USB_A, J3 Conn_01x07_Pin, U1 RP2040, U2 NCP1117ST33T3G, U3 W25Q128JVSIM, X1 SW_Omron_B3FS-1000P, Y1 ABM8-272-T3, Y2 SW_Omron_B3FS-1000P

Commit message: update usb A connector
Parts:
- J2: value USB_A -> USB1046-GF-0190-L-B
Changed lines of the file:
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@@
 			)
 		)
-		(property "Value" "USB_A"
+		(property "Value" "USB1046-GF-0190-L-B"
 			(at 0 -8.5 0)
 			(layer "B.Fab")
@@
 			)
 		)
-		(property "Datasheet" "https://mm.digikey.com/Volume0/opasdata/d220001/medias/docus/5335/USB1046_Spec.pdf"
+		(property "Datasheet" "https://gct.co/connector/usb1046"
 			(at 0 0 0)
 			(unlocked yes)
@@
 			)
 		)
-		(property "Description" "USB Type A connector"
+		(property "Description" "USB Type A connector GCT USB1046-GF-0190-L-B"
 			(at 0 0 0)
 			(unlocked yes)
